Commit message: feat(quadruped_description): add collision geometry

File: quadruped_description/urdf/quadruped_description.urdf (robot description, URDF)
Before this commit: robot quadruped_description, 13 links, 12 joints
Links:
- link base_link: geometry collision mesh filename=package://quadruped_description/meshes/collision/base_link.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; visual mesh filename=package://quadruped_description/meshes/visual/base_link.STL
- link hip_fl_link: geometry collision mesh filename=package://quadruped_description/meshes/collision/hip_fl_lin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; visual mesh filename=package://quadruped_description/meshes/visual/hip_fl_link.S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
- link hip_fr_link: geometry collision mesh filename=package://quadruped_description/meshes/collision/hip_fr_lin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; visual mesh filename=package://quadruped_description/meshes/visual/hip_fr_link.S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
- link hip_rl_link: geometry collision mesh filename=package://quadruped_description/meshes/collision/hip_rl_lin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; visual mesh filename=package://quadruped_description/meshes/visual/hip_rl_link.S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
- link hip_rr_link: geometry collision mesh filename=package://quadruped_description/meshes/collision/hip_rr_lin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; visual mesh filename=package://quadruped_description/meshes/visual/hip_rr_link.S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
- link shank_fl_link: geometry collision mesh filename=package://quadruped_description/meshes/collision/shank_fl_l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; visual mesh filename=package://quadruped_description/meshes/visual/shank_fl_link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
- link shank_fr_link: geometry collision mesh filename=package://quadruped_description/meshes/collision/shank_fr_l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; visual mesh filename=package://quadruped_description/meshes/visual/shank_fr_link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
- link shank_rl_link: geometry collision mesh filename=package://quadruped_description/meshes/collision/shank_rl_l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; visual mesh filename=package://quadruped_description/meshes/visual/shank_rl_link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
- link shank_rr_link: geometry collision mesh filename=package://quadruped_description/meshes/collision/shank_rr_l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; visual mesh filename=package://quadruped_description/meshes/visual/shank_rr_link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
- link thigh_fl_link: geometry collision mesh filename=package://quadruped_description/meshes/collision/thigh_fl_l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; visual mesh filename=package://quadruped_description/meshes/visual/thigh_fl_link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
- link thigh_fr_link: geometry collision mesh filename=package://quadruped_description/meshes/collision/thigh_fr_l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; visual mesh filename=package://quadruped_description/meshes/visual/thigh_fr_link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
- link thigh_rl_link: geometry collision mesh filename=package://quadruped_description/meshes/collision/thigh_rl_l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; visual mesh filename=package://quadruped_description/meshes/visual/thigh_rl_link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
- link thigh_rr_link: geometry collision mesh filename=package://quadruped_description/meshes/collision/thigh_rr_l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; visual mesh filename=package://quadruped_description/meshes/visual/thigh_rr_link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
